File: hardware/vallox-rs485-controller.kicad_sch (KiCad schematic)
At the start: 60 parts, among them J1 + - A B M, J2 TYPE-C-31-M-12, J3 HS20HS072RX, Q1 AO3400A, SW1 -, SW2 +, SW3 OK, SW4 BACK, U1 ESP32-C3-WROOM-02-N4, U2 TPS54202DDC, U3 ME6211C33M5G-N, U4 THVD1400DR

Commit message: hw(pcb): rev A placement on a 104 x 66 mm board, not yet routed
The board file was empty. All 60 schematic parts are now on the top side,
placed from the netlist with KiCad's bundled pcbnew Python (KiCad closed):
the MCP server had no pcb_write tools this session and the file-based MCP
transfer tool is the one the workspace forbids. Every footprint carries its
symbol UUID as path, so a GUI F8 should reconcile to no changes.

Floor plan: display glass reserve top-left with the four buttons centred
under it and the LEDs beside it; FPC connector on the glass's short edge;
ESP32 module top-right with its antenna 6 mm over the edge, the position the
Espressif hardware design guide recommends; terminal block and USB-C flush
with the right edge so all field wiring enters from one wall; buck in the
bottom-right corner, RS-485 front end between terminal and module.

kicad-cli drc --severity-all --schematic-parity: 0 errors, 7 warnings
(silkscreen of edge-mounted U1/J1/J2 crossing the edge; U1 thermal vias
widened from 0.2 to 0.3 mm drill to meet the project's min-hole rule),
parity clean apart from the four intentional mounting holes, 138 unconnected
items because nothing is routed. Parity caught two build mistakes on the way:
footprints written without their library nickname, and TP1/TP2/JP1 symbols
not excluded from BOM while their footprints are — the symbols now say
in_bom no, ERC unchanged.

CI's DRC step will stay red on this branch until the board is routed:
--exit-code-violations also counts unconnected items (verified locally).
Parts:
- JP1, TP1, TP2: now left out of the parts list
Changed lines of the file:
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@@
 		(unit 1)
 		(exclude_from_sim no)
-		(in_bom yes)
+		(in_bom no)
 		(on_board yes)
 		(dnp no)
@@
 		(unit 1)
 		(exclude_from_sim no)
-		(in_bom yes)
+		(in_bom no)
 		(on_board yes)
 		(dnp no)
@@
 		(unit 1)
 		(exclude_from_sim no)
-		(in_bom yes)
-		(on_board yes)
-		(dnp no)
+		(in_bom no)
+		(on_board yes)
+		(dnp no)

Commit message: hw(display): straight tail into a top-contact FH12A; J3 mirrored in the schematic
The fold would have lifted the FPC loop above the glass and cost a manual
step per unit. With the contact side known, a top-contact connector takes
the tail straight: Hirose FH12A-12S-0.5SH(55) shares the FH12 land pattern
(catalogue p. 10), so the footprint and model stay; J3 moves east so its
entry face is 16.9 mm from the glass edge and DS1 carries the straight model.

Straight insertion puts tail contact k on the pad the footprint numbers
13-k — a fact of coordinates, verified on the board (pad 11 = CS meets
contact 2 at y 28.17) — so the schematic symbol is mirrored and the mapping
written out pin by pin. ERC unchanged, netlist checked, board pad nets
re-synced, DRC 0 errors / 7 known warnings, schematic parity clean.
Parts:
- J3: value HS20HS072RX -> FH12A-12S-0.5SH(55); LCSC (none) -> C596811; MPN (none) -> FH12A-12S-0.5SH(55); Manufacturer (none) -> Hirose
Connections:
- net +3V3: now also J3.4 (Pin_4), J3.5 (Pin_5); no longer J3.8 (Pin_8), J3.9 (Pin_9)
- net TFT_CS: now also J3.11 (Pin_11); no longer J3.2 (Pin_2)
- net TFT_DC: now also J3.10 (Pin_10); no longer J3.3 (Pin_3)
- net TFT_LED_K: now also J3.2 (Pin_2); no longer J3.11 (Pin_11)
- net TFT_MOSI: now also J3.8 (Pin_8); no longer J3.5 (Pin_5)
- net TFT_RST: now also J3.7 (Pin_7); no longer J3.6 (Pin_6)
- net TFT_SCK: now also J3.9 (Pin_9); no longer J3.4 (Pin_4)
- net at R11.2: now also J3.3 (Pin_3); no longer J3.10 (Pin_10)
Other:
- note added: "J3 = FH12A top-contact; display tail straight, contacts up. Tail contact k meets J3 pad 13-k, so the symbol is mirrored: J3 pin 1 = display 12 (GND) ... J3 pin 12 = display 1 (GND)."
Changed lines of the file:
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@@
 		(comment 4 "Power stage provisional until measurements M1/M2a")
+	)
+	(text "J3 = FH12A top-contact; display tail straight, contacts up.\nTail contact k meets J3 pad 13-k, so the symbol is mirrored:\nJ3 pin 1 = display 12 (GND) ... J3 pin 12 = display 1 (GND)."
+		(exclude_from_sim no)
+		(at 226.06 69.85 0)
+		(effects (font (size 1.27 1.27)) (justify left bottom))
 	)
 	(symbol
@@
 	(symbol
 		(lib_id "Connector_Generic:Conn_01x12")
-		(at 215.9 93.98 180)
+		(at 215.9 91.44 180)
+		(mirror x)
 		(unit 1)
 		(exclude_from_sim no)
@@
 			(effects (font (size 1.27 1.27)))
 		)
-		(property "Value" "HS20HS072RX"
+		(property "Value" "FH12A-12S-0.5SH(55)"
 			(at 215.9 97.79 180)
 			(effects (font (size 1.27 1.27)))
@@
 			(at 215.9 93.98 0)
 			(effects (font (size 1.27 1.27)) (hide yes))
+		)		(property "Manufacturer" "Hirose"
+			(at 215.9 93.98 0)
+			(effects (font (size 1.27 1.27)) (hide yes))
+		)
+		(property "MPN" "FH12A-12S-0.5SH(55)"
+			(at 215.9 93.98 0)
+			(effects (font (size 1.27 1.27)) (hide yes))
+		)
+		(property "LCSC" "C596811"
+			(at 215.9 93.98 0)
+			(effects (font (size 1.27 1.27)) (hide yes))
+		)
+		(property "Description" "0.5 mm 12-pin FPC connector, TOP contact, for the display tail inserted straight with its contacts up; J3 pin k carries display pin 13-k (symbol mirrored)"
+			(at 215.9 93.98 0)
+			(effects (font (size 1.27 1.27)) (hide yes))

Commit message: hw(bom): every schematic line carries Manufacturer, MPN and LCSC; R5-R7 get the DNP attribute
The order gate reads the schematic, so the schematic has to be the bill of
materials. 56 lines had only value and footprint; each code was checked
against the JLCPCB catalogue today (MPN, package, stock, Basic/Extended) and
the list is kept as hardware/docs/parts-revA.csv, the file the fields were
written from.

Three things were decided on the way and are in decisions.md: the indicator
LEDs must be low-Vf types because 3.3 V through 1 k does not light an InGaN
green (PWR yellow-green, BUS yellow, FAULT red); J1 is the Dorabo
DB128V-5.08-5P (no 5-pole Phoenix MKDS in the catalogue); L1 is the 22 uH
FNR6045S220MT the schematic already called for. R4 13.3 k stays Extended
rather than drifting the 5 V rail to a Basic value.

Title block: the power stage is no longer provisional (M1/M2a measured).
Parts:
- C1: LCSC (none) -> C136294; MPN (none) -> UCD1V221MNL1GS; Manufacturer (none) -> Nichicon
- C10, C7: LCSC (none) -> C19702; MPN (none) -> CL10A106KP8NNNC; Manufacturer (none) -> Samsung Electro-Mechanics
- C11, C12, C3, C8: LCSC (none) -> C14663; MPN (none) -> CC0603KRX7R9BB104; Manufacturer (none) -> YAGEO
- C13, C9: LCSC (none) -> C15849; MPN (none) -> CL10A105KB8NNNC; Manufacturer (none) -> Samsung Electro-Mechanics
- C2: LCSC (none) -> C377773; MPN (none) -> CL21A225KBQNNNE; Manufacturer (none) -> Samsung Electro-Mechanics
- C4, C5: LCSC (none) -> C45783; MPN (none) -> CL21A226MAQNNNE; Manufacturer (none) -> Samsung Electro-Mechanics
- D1, D3: LCSC (none) -> C8678; MPN (none) -> SS34; Manufacturer (none) -> MDD
- D2: LCSC (none) -> C32677; MPN (none) -> PSM712-LF-T7; Manufacturer (none) -> ProTek Devices
- D4: LCSC (none) -> C965805; MPN (none) -> XL-1608SYGC-06; Manufacturer (none) -> XINGLIGHT
- D5: LCSC (none) -> C2286; MPN (none) -> KT-0603R; Manufacturer (none) -> Hongli Zhihui
- D6: LCSC (none) -> C84268; MPN (none) -> NCD0603Y1; Manufacturer (none) -> Nationstar
- F1, F2: LCSC (none) -> C1884489; MPN (none) -> JK-mSMD010-60; Manufacturer (none) -> JK
- J1: LCSC (none) -> C2927513; MPN (none) -> DB128V-5.08-5P-GN-S; Manufacturer (none) -> Dorabo
- J2: LCSC (none) -> C165948; MPN (none) -> TYPE-C-31-M-12; Manufacturer (none) -> Korean Hroparts Elec
- L1: LCSC (none) -> C168080; MPN (none) -> FNR6045S220MT; Manufacturer (none) -> Changjiang Microelectronics
- Q1: LCSC (none) -> C20917; MPN (none) -> AO3400A; Manufacturer (none) -> Alpha & Omega Semiconductor
- R1, R3: LCSC (none) -> C25803; MPN (none) -> 0603WAF1003T5E; Manufacturer (none) -> UNI-ROYAL
- R10, R13, R19, R21, R22, R8, R9: LCSC (none) -> C25804; MPN (none) -> 0603WAF1002T5E; Manufacturer (none) -> UNI-ROYAL
- R11: LCSC (none) -> C17946; MPN (none) -> 1206W4F270JT5E; Manufacturer (none) -> UNI-ROYAL
- R12: LCSC (none) -> C22775; MPN (none) -> 0603WAF1000T5E; Manufacturer (none) -> UNI-ROYAL
- R14, R15: LCSC (none) -> C23186; MPN (none) -> 0603WAF5101T5E; Manufacturer (none) -> UNI-ROYAL
- R2: LCSC (none) -> C22809; MPN (none) -> 0603WAF1502T5E; Manufacturer (none) -> UNI-ROYAL
- R20, R26, R27: LCSC (none) -> C21190; MPN (none) -> 0603WAF1001T5E; Manufacturer (none) -> UNI-ROYAL
- R23: LCSC (none) -> C22843; MPN (none) -> 0603WAF1501T5E; Manufacturer (none) -> UNI-ROYAL
- R24: LCSC (none) -> C22978; MPN (none) -> 0603WAF3301T5E; Manufacturer (none) -> UNI-ROYAL
- R25: LCSC (none) -> C23212; MPN (none) -> 0603WAF6801T5E; Manufacturer (none) -> UNI-ROYAL
- R4: LCSC (none) -> C25952; MPN (none) -> 0603WAF1332T5E; Manufacturer (none) -> UNI-ROYAL
- R5: LCSC (none) -> C22787; MPN (none) -> 0603WAF1200T5E; Manufacturer (none) -> UNI-ROYAL; now not fitted
- R6, R7: LCSC (none) -> C21190; MPN (none) -> 0603WAF1001T5E; Manufacturer (none) -> UNI-ROYAL; now not fitted
- SW1, SW2, SW3, SW4: LCSC (none) -> C221880; MPN (none) -> PTS645SM43SMTR92LFS; Manufacturer (none) -> C&K
- U1: LCSC (none) -> C2934560; MPN (none) -> ESP32-C3-WROOM-02-N4; Manufacturer (none) -> Espressif Systems
- U2: LCSC (none) -> C191884; MPN (none) -> TPS54202DDCR; Manufacturer (none) -> Texas Instruments
- U3: LCSC (none) -> C82942; MPN (none) -> ME6211C33M5G-N; Manufacturer (none) -> Microne
- U4: LCSC (none) -> C3235232; MPN (none) -> THVD1400DR; Manufacturer (none) -> Texas Instruments
