File: hardware/vallox-rs485-controller.kicad_sch (KiCad schematic)
At the start: 0 parts

Commit message: hw(sch): rev A schematic, drawn as continuous wires on one A3 sheet
Drawn ahead of the rail measurements at Miro's request, so that there is
something concrete to review. The power stage is marked provisional in the
title block; what M1/M2a can still change is listed in decisions.md and is
contained in the power region.

Every connection is a wire from pin to pin. Local labels only name nets; they
never carry a connection. Power rails use power symbols. ERC with kicad-cli
10.0.2: 0 errors, 1 warning (Q1's embedded symbol differs from the library
copy - cosmetic). Netlist: 47 nets, the only single-node nets are the four
intentional no-connects.

Decisions made while drawing, each with its datasheet page in decisions.md:
5 V intermediate rail with a 3.3 V LDO so the backlight and USB bench power
have a clean path; 22 uH instead of 10 uH from the ripple arithmetic; EN
divider because the pin's absolute maximum is 7 V; the GPIO map chosen so
that wires do not cross, with the button ladder on IO4 because IO0-IO4 are
the only ADC1 pins; the display tail is 12-pin, not 30 as the candidate list
had it.

Two tool facts cost time and are recorded in layout-notes.md: pins landing
on a wire's interior need explicit junctions (52 added), and the pin-position
tool reports rotation 90 mirrored relative to KiCad - the VBUS diode was
drawn backwards until the netlist said so. J1 and U4 are mirrored in the
file because no tool does it.
Parts:
- added C1: 220u/35V, Capacitor_SMD:CP_Elec_8x10.5, symbol Device:C_Polarized
- added C10, C7: 10u, Capacitor_SMD:C_0603_1608Metric, symbol Device:C
- added C11, C12, C3, C8: 100n, Capacitor_SMD:C_0603_1608Metric, symbol Device:C
- added C13, C9: 1u, Capacitor_SMD:C_0603_1608Metric, symbol Device:C
- added C2: 2.2u/50V, Capacitor_SMD:C_0805_2012Metric, symbol Device:C
- added C4, C5: 22u/10V, Capacitor_SMD:C_0805_2012Metric, symbol Device:C
- added D1, D3: SS34, Diode_SMD:D_SMA, symbol Device:D_Schottky
- added D2: SM712, Package_TO_SOT_SMD:SOT-23, symbol Diode:SM712_SOT23
- added D4: PWR, LED_SMD:LED_0603_1608Metric, symbol Device:LED
- added D5: FAULT, LED_SMD:LED_0603_1608Metric, symbol Device:LED
- added D6: BUS, LED_SMD:LED_0603_1608Metric, symbol Device:LED
- added F1, F2: 100mA/60V, Fuse:Fuse_1812_4532Metric, symbol Device:Polyfuse
- added J1: + - A B M, TerminalBlock_Phoenix:TerminalBlock_Phoenix_MKDS-1,5-5-5.08_1x05_P5.08mm_Horizontal, symbol Connector:Screw_Terminal_01x05
- added J2: TYPE-C-31-M-12, Connector_USB:USB_C_Receptacle_HRO_TYPE-C-31-M-12, symbol Connector:USB_C_Receptacle_USB2.0_16P
- added J3: HS20HS072RX, Connector_FFC-FPC:Hirose_FH12-12S-0.5SH_1x12-1MP_P0.50mm_Horizontal, symbol Connector_Generic:Conn_01x12
- added JP1: TERM, Jumper:SolderJumper-2_P1.3mm_Open_RoundedPad1.0x1.5mm, symbol Jumper:SolderJumper_2_Open
- added L1: 22uH, Inductor_SMD:L_Changjiang_FNR6045S, symbol Device:L
- added Q1: AO3400A, Package_TO_SOT_SMD:SOT-23, symbol Transistor_FET:AO3400A
- added R1, R3: 100k, Resistor_SMD:R_0603_1608Metric, symbol Device:R
- added R10, R13, R19, R21, R22, R8, R9: 10k, Resistor_SMD:R_0603_1608Metric, symbol Device:R
- added R11: 27R, Resistor_SMD:R_1206_3216Metric, symbol Device:R
- added R12: 100R, Resistor_SMD:R_0603_1608Metric, symbol Device:R
- added R14, R15: 5.1k, Resistor_SMD:R_0603_1608Metric, symbol Device:R
- added R2: 15k, Resistor_SMD:R_0603_1608Metric, symbol Device:R
- added R20, R26, R27: 1k, Resistor_SMD:R_0603_1608Metric, symbol Device:R
- added R23: 1.5k, Resistor_SMD:R_0603_1608Metric, symbol Device:R
- added R24: 3.3k, Resistor_SMD:R_0603_1608Metric, symbol Device:R
- added R25: 6.8k, Resistor_SMD:R_0603_1608Metric, symbol Device:R
- added R4: 13.3k, Resistor_SMD:R_0603_1608Metric, symbol Device:R
- added R5: 120R DNP, Resistor_SMD:R_0603_1608Metric, symbol Device:R
- added R6, R7: 1k DNP, Resistor_SMD:R_0603_1608Metric, symbol Device:R
- added SW1: -, Button_Switch_SMD:SW_SPST_PTS645Sx43SMTR92, symbol Switch:SW_Push
- added SW2: +, Button_Switch_SMD:SW_SPST_PTS645Sx43SMTR92, symbol Switch:SW_Push
- added SW3: OK, Button_Switch_SMD:SW_SPST_PTS645Sx43SMTR92, symbol Switch:SW_Push
- added SW4: BACK, Button_Switch_SMD:SW_SPST_PTS645Sx43SMTR92, symbol Switch:SW_Push
- added TP1: EN, TestPoint:TestPoint_Pad_1.0x1.0mm, symbol Connector:TestPoint
- added TP2: BOOT, TestPoint:TestPoint_Pad_1.0x1.0mm, symbol Connector:TestPoint
- added U1: ESP32-C3-WROOM-02-N4, RF_Module:ESP32-C3-WROOM-02, symbol RF_Module:ESP32-C3-WROOM-02
- added U2: TPS54202DDC, Package_TO_SOT_SMD:SOT-23-6, symbol Regulator_Switching:TPS54202DDC
- added U3: ME6211C33M5G-N, Package_TO_SOT_SMD:SOT-23-5, symbol Regulator_Linear:ME6211C33M5
- added U4: THVD1400DR, Package_SO:SOIC-8_3.9x4.9mm_P1.27mm, symbol Interface_UART:THVD1400D
Connections:
- new net: R3.1, R4.1, U2.4 (FB)
- new net: R24.1, SW3.1
- new net: J3.10 (Pin_10), R11.2
- new net: R25.1, SW4.1
- new net: J2.B5 (CC2), R15.1
- new net: J2.A5 (CC1), R14.1
- new net: R1.2, R2.1, U2.5 (EN)
- new net: D4.2 (A), R20.1
- new net: F1.1, J1.3 (Pin_3)
- new net: F2.1, J1.4 (Pin_4)
- new net: R27.1, U1.11 (IO20/RXD)
- new net: D6.2 (A), R27.2
- new net: C3.1, U2.6 (BOOT)
- new net: Q1.1 (G), R12.2, R13.1
- new net: R23.1, SW2.1
- new net: C13.1, R19.2, TP1.1, U1.2 (EN)
- new net: R20.2, U1.4 (IO5)
- new net: JP1.2 (B), R5.2
- new net: D5.2 (A), R26.1
- new net: R26.2, U1.10 (IO10)
- new net: TP2.1, U1.8 (IO9)
- new net +3V3: C10.1, C11.1, C7.1, C8.1, J3.8 (Pin_8), J3.9 (Pin_9), R10.1, R19.1, R21.1, R22.1, R6.1, R9.2, U1.1 (3V3), U3.5 (V_{OUT}), U4.8 (VCC)
- new net +5V: C4.1, C5.1, D3.1 (K), L1.2, R11.1, R3.2, U3.1 (V_{IN}), U3.3 (CE)
- new net BTN_ADC: C12.1, R22.2, SW1.2, SW2.2, SW3.2, SW4.2, U1.3 (IO4)
- new net GND: C1.2, C10.2, C11.2, C12.2, C13.2, C2.2, C4.2, C5.2, C7.2, C8.2, C9.2, D2.3 (common), D4.1 (K), D5.1 (K), D6.1 (K), J1.2 (Pin_2), J1.5 (Pin_5), J2.A1 (GND), J2.A12 (GND), J2.B1 (GND), J2.B12 (GND), J2.SH (SHIELD), J3.1 (Pin_1), J3.12 (Pin_12), Q1.2 (S), R13.2, R14.2, R15.2, R2.2, R23.2, R24.2, R25.2, R4.2, R7.2, R8.2, SW1.1, U1.19 (GND), U1.9 (GND), U2.1 (GND), U3.2 (V_{SS}), U4.5 (GND)
- new net PANEL_21V: D1.2 (A), J1.1 (Pin_1)
- new net RS485_A: D2.2 (A2), F1.2, R5.1, R6.2, U4.6 (A)
- new net RS485_B: D2.1 (A1), F2.2, JP1.1 (A), R7.1, U4.7 (B)
- new net RS485_DE: R8.1, U1.6 (IO7), U4.2 (~{RE}), U4.3 (DE)
- new net RS485_RX: U1.5 (IO6), U4.1 (RO)
- new net RS485_TX: R9.1, U1.7 (IO8), U4.4 (DI)
- new net SW: C3.2, L1.1, U2.2 (SW)
- new net TFT_BL_PWM: R12.1, U1.12 (IO21/TXD)
- new net TFT_CS: J3.2 (Pin_2), U1.15 (IO3)
- new net TFT_DC: J3.3 (Pin_3), R21.2, U1.16 (IO2)
- new net TFT_LED_K: J3.11 (Pin_11), Q1.3 (D)
- new net TFT_MOSI: J3.5 (Pin_5), U1.18 (IO0)
- new net TFT_RST: C9.1, J3.6 (Pin_6), R10.2
- new net TFT_SCK: J3.4 (Pin_4), U1.17 (IO1)
- new net USB_D+: J2.A6 (D+), J2.B6 (D+), U1.14 (IO19)
- new net USB_D-: J2.A7 (D-), J2.B7 (D-), U1.13 (IO18)
- new net VBUS: D3.2 (A), J2.A4 (VBUS), J2.A9 (VBUS), J2.B4 (VBUS), J2.B9 (VBUS)
- new net VIN_BUCK: C1.1, C2.1, D1.1 (K), R1.1, U2.3 (VIN)
- no-connect marks 0 -> 4

Commit message: hw(pcb): rev A placed, routed and sourced (#6)
* hw(pcb): rev A placement on a 104 x 66 mm board, not yet routed

The board file was empty. All 60 schematic parts are now on the top side,
placed from the netlist with KiCad's bundled pcbnew Python (KiCad closed):
the MCP server had no pcb_write tools this session and the file-based MCP
transfer tool is the one the workspace forbids. Every footprint carries its
symbol UUID as path, so a GUI F8 should reconcile to no changes.

Floor plan: display glass reserve top-left with the four buttons centred
under it and the LEDs beside it; FPC connector on the glass's short edge;
ESP32 module top-right with its antenna 6 mm over the edge, the position the
Espressif hardware design guide recommends; terminal block and USB-C flush
with the right edge so all field wiring enters from one wall; buck in the
bottom-right corner, RS-485 front end between terminal and module.

kicad-cli drc --severity-all --schematic-parity: 0 errors, 7 warnings
(silkscreen of edge-mounted U1/J1/J2 crossing the edge; U1 thermal vias
widened from 0.2 to 0.3 mm drill to meet the project's min-hole rule),
parity clean apart from the four intentional mounting holes, 138 unconnected
items because nothing is routed. Parity caught two build mistakes on the way:
footprints written without their library nickname, and TP1/TP2/JP1 symbols
not excluded from BOM while their footprints are — the symbols now say
in_bom no, ERC unchanged.

CI's DRC step will stay red on this branch until the board is routed:
--exit-code-violations also counts unconnected items (verified locally).

* docs(display): tail geometry verified from the HSD drawing; contact side still open

The placement assumed the FPC tail leaves the short edge toward J3. The
manufacturer drawing confirms edge, centring and a 20.7 mm length, and adds
the consequence: the tail bends, a bend flips the contact side, and the
drawing does not state the contact side unambiguously. J3's orientation
depends on it, s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
Parts:
- C1: LCSC (none) -> C136294; MPN (none) -> UCD1V221MNL1GS; Manufacturer (none) -> Nichicon
- C10, C7: LCSC (none) -> C19702; MPN (none) -> CL10A106KP8NNNC; Manufacturer (none) -> Samsung Electro-Mechanics
- C11, C12, C3, C8: LCSC (none) -> C14663; MPN (none) -> CC0603KRX7R9BB104; Manufacturer (none) -> YAGEO
- C13, C9: LCSC (none) -> C15849; MPN (none) -> CL10A105KB8NNNC; Manufacturer (none) -> Samsung Electro-Mechanics
- C2: LCSC (none) -> C377773; MPN (none) -> CL21A225KBQNNNE; Manufacturer (none) -> Samsung Electro-Mechanics
- C4, C5: LCSC (none) -> C45783; MPN (none) -> CL21A226MAQNNNE; Manufacturer (none) -> Samsung Electro-Mechanics
- D1, D3: LCSC (none) -> C8678; MPN (none) -> SS34; Manufacturer (none) -> MDD
- D2: LCSC (none) -> C32677; MPN (none) -> PSM712-LF-T7; Manufacturer (none) -> ProTek Devices
- D4: LCSC (none) -> C965805; MPN (none) -> XL-1608SYGC-06; Manufacturer (none) -> XINGLIGHT
- D5: LCSC (none) -> C2286; MPN (none) -> KT-0603R; Manufacturer (none) -> Hongli Zhihui
- D6: LCSC (none) -> C84268; MPN (none) -> NCD0603Y1; Manufacturer (none) -> Nationstar
- F1, F2: LCSC (none) -> C1884489; MPN (none) -> JK-mSMD010-60; Manufacturer (none) -> JK
- J1: LCSC (none) -> C2927513; MPN (none) -> DB128V-5.08-5P-GN-S; Manufacturer (none) -> Dorabo
- J2: LCSC (none) -> C165948; MPN (none) -> TYPE-C-31-M-12; Manufacturer (none) -> Korean Hroparts Elec
- J3: value HS20HS072RX -> FH12A-12S-0.5SH(55); LCSC (none) -> C596811; MPN (none) -> FH12A-12S-0.5SH(55); Manufacturer (none) -> Hirose
- JP1, TP1, TP2: now left out of the parts list
- L1: LCSC (none) -> C168080; MPN (none) -> FNR6045S220MT; Manufacturer (none) -> Changjiang Microelectronics
- Q1: LCSC (none) -> C20917; MPN (none) -> AO3400A; Manufacturer (none) -> Alpha & Omega Semiconductor
- R1, R3: LCSC (none) -> C25803; MPN (none) -> 0603WAF1003T5E; Manufacturer (none) -> UNI-ROYAL
- R10, R13, R19, R21, R22, R8, R9: LCSC (none) -> C25804; MPN (none) -> 0603WAF1002T5E; Manufacturer (none) -> UNI-ROYAL
- R11: LCSC (none) -> C17946; MPN (none) -> 1206W4F270JT5E; Manufacturer (none) -> UNI-ROYAL
- R12: LCSC (none) -> C22775; MPN (none) -> 0603WAF1000T5E; Manufacturer (none) -> UNI-ROYAL
- R14, R15: LCSC (none) -> C23186; MPN (none) -> 0603WAF5101T5E; Manufacturer (none) -> UNI-ROYAL
- R2: LCSC (none) -> C22809; MPN (none) -> 0603WAF1502T5E; Manufacturer (none) -> UNI-ROYAL
- R20, R26, R27: LCSC (none) -> C21190; MPN (none) -> 0603WAF1001T5E; Manufacturer (none) -> UNI-ROYAL
- R23: LCSC (none) -> C22843; MPN (none) -> 0603WAF1501T5E; Manufacturer (none) -> UNI-ROYAL
- R24: LCSC (none) -> C22978; MPN (none) -> 0603WAF3301T5E; Manufacturer (none) -> UNI-ROYAL
- R25: LCSC (none) -> C23212; MPN (none) -> 0603WAF6801T5E; Manufacturer (none) -> UNI-ROYAL
- R4: LCSC (none) -> C25952; MPN (none) -> 0603WAF1332T5E; Manufacturer (none) -> UNI-ROYAL
- R5: LCSC (none) -> C22787; MPN (none) -> 0603WAF1200T5E; Manufacturer (none) -> UNI-ROYAL; now not fitted
- R6, R7: LCSC (none) -> C21190; MPN (none) -> 0603WAF1001T5E; Manufacturer (none) -> UNI-ROYAL; now not fitted
- SW1, SW2, SW3, SW4: LCSC (none) -> C221880; MPN (none) -> PTS645SM43SMTR92LFS; Manufacturer (none) -> C&K
- U1: LCSC (none) -> C2934560; MPN (none) -> ESP32-C3-WROOM-02-N4; Manufacturer (none) -> Espressif Systems
- U2: LCSC (none) -> C191884; MPN (none) -> TPS54202DDCR; Manufacturer (none) -> Texas Instruments
- U3: LCSC (none) -> C82942; MPN (none) -> ME6211C33M5G-N; Manufacturer (none) -> Microne
- U4: LCSC (none) -> C3235232; MPN (none) -> THVD1400DR; Manufacturer (none) -> Texas Instruments
Connections:
- net +3V3: now also J3.4 (Pin_4), J3.5 (Pin_5); no longer J3.8 (Pin_8), J3.9 (Pin_9)
- net TFT_CS: now also J3.11 (Pin_11); no longer J3.2 (Pin_2)
- net TFT_DC: now also J3.10 (Pin_10); no longer J3.3 (Pin_3)
- net TFT_LED_K: now also J3.2 (Pin_2); no longer J3.11 (Pin_11)
- net TFT_MOSI: now also J3.8 (Pin_8); no longer J3.5 (Pin_5)
- net TFT_RST: now also J3.7 (Pin_7); no longer J3.6 (Pin_6)
- net TFT_SCK: now also J3.9 (Pin_9); no longer J3.4 (Pin_4)
- net at R11.2: now also J3.3 (Pin_3); no longer J3.10 (Pin_10)
Other:
- note added: "J3 = FH12A top-contact; display tail straight, contacts up. Tail contact k meets J3 pad 13-k, so the symbol is mirrored: J3 pin 1 = display 12 (GND) ... J3 pin 12 = display 1 (GND)."
