File: hardware/vallox-rs485-controller.kicad_pcb (KiCad board)
At the start: 0 parts

Commit message: hw(pcb): rev A placed, routed and sourced (#6)
* hw(pcb): rev A placement on a 104 x 66 mm board, not yet routed

The board file was empty. All 60 schematic parts are now on the top side,
placed from the netlist with KiCad's bundled pcbnew Python (KiCad closed):
the MCP server had no pcb_write tools this session and the file-based MCP
transfer tool is the one the workspace forbids. Every footprint carries its
symbol UUID as path, so a GUI F8 should reconcile to no changes.

Floor plan: display glass reserve top-left with the four buttons centred
under it and the LEDs beside it; FPC connector on the glass's short edge;
ESP32 module top-right with its antenna 6 mm over the edge, the position the
Espressif hardware design guide recommends; terminal block and USB-C flush
with the right edge so all field wiring enters from one wall; buck in the
bottom-right corner, RS-485 front end between terminal and module.

kicad-cli drc --severity-all --schematic-parity: 0 errors, 7 warnings
(silkscreen of edge-mounted U1/J1/J2 crossing the edge; U1 thermal vias
widened from 0.2 to 0.3 mm drill to meet the project's min-hole rule),
parity clean apart from the four intentional mounting holes, 138 unconnected
items because nothing is routed. Parity caught two build mistakes on the way:
footprints written without their library nickname, and TP1/TP2/JP1 symbols
not excluded from BOM while their footprints are — the symbols now say
in_bom no, ERC unchanged.

CI's DRC step will stay red on this branch until the board is routed:
--exit-code-violations also counts unconnected items (verified locally).

* docs(display): tail geometry verified from the HSD drawing; contact side still open

The placement assumed the FPC tail leaves the short edge toward J3. The
manufacturer drawing confirms edge, centring and a 20.7 mm length, and adds
the consequence: the tail bends, a bend flips the contact side, and the
drawing does not state the contact side unambiguously. J3's orientation
depends on it, s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
Parts:
- added C1: 220u/35V, Capacitor_SMD:CP_Elec_8x10.5, F.Cu at (80.0, 58.5)
- added C10: 10u, Capacitor_SMD:C_0603_1608Metric, F.Cu at (80.3, 2.20)
- added C11: 100n, Capacitor_SMD:C_0603_1608Metric, F.Cu at (75.5, 2.20)
- added C12: 100n, Capacitor_SMD:C_0603_1608Metric, F.Cu at (80.3, 13.4)
- added C13: 1u, Capacitor_SMD:C_0603_1608Metric, F.Cu at (80.3, 7.80)
- added C2: 2.2u/50V, Capacitor_SMD:C_0805_2012Metric, F.Cu at (79.8, 50.2)
- added C3: 100n, Capacitor_SMD:C_0603_1608Metric, F.Cu at (85.6, 47.6)
- added C4: 22u/10V, Capacitor_SMD:C_0805_2012Metric, F.Cu at (69.0, 48.6)
- added C5: 22u/10V, Capacitor_SMD:C_0805_2012Metric, F.Cu at (69.0, 52.2)
- added C7: 10u, Capacitor_SMD:C_0603_1608Metric, F.Cu at (72.8, 42.5)
- added C8: 100n, Capacitor_SMD:C_0603_1608Metric, F.Cu at (84.8, 38.6)
- added C9: 1u, Capacitor_SMD:C_0603_1608Metric, F.Cu at (86.0, 23.5)
- added D1: SS34, Diode_SMD:D_SMA, F.Cu at (89.9, 59.5)
- added D2: SM712, Package_TO_SOT_SMD:SOT-23, F.Cu at (90.8, 36.0)
- added D3: SS34, Diode_SMD:D_SMA, F.Cu at (89.5, 32.4)
- added D4: PWR, LED_SMD:LED_0603_1608Metric, F.Cu at (63.8, 7.80)
- added D5: FAULT, LED_SMD:LED_0603_1608Metric, F.Cu at (63.8, 13.8)
- added D6: BUS, LED_SMD:LED_0603_1608Metric, F.Cu at (63.8, 10.8)
- added DS1: HS20HS072RX, mironet:LCD_2.0in_HSD_HS20HS072RX_FPC-12P-0.5mm, F.Cu at (33.9, 26.1)
- added F1: 100mA/60V, Fuse:Fuse_1812_4532Metric, F.Cu at (90.2, 45.6)
- added F2: 100mA/60V, Fuse:Fuse_1812_4532Metric, F.Cu at (90.2, 39.9)
- added H1: M3, MountingHole:MountingHole_3.2mm_M3, F.Cu at (3.50, 3.50)
- added H2: M3, MountingHole:MountingHole_3.2mm_M3, F.Cu at (3.50, 62.5)
- added H3: M3, MountingHole:MountingHole_3.2mm_M3, F.Cu at (100.5, 62.5)
- added H4: M3, MountingHole:MountingHole_3.2mm_M3, F.Cu at (66.0, 3.50)
- added J1: + - A B M, TerminalBlock_Phoenix:TerminalBlock_Phoenix_MKDS-1,5-5-5.08_1x05_P5.08mm_Horizontal, F.Cu at (99.4, 55.5)
- added J2: TYPE-C-31-M-12, Connector_USB:USB_C_Receptacle_HRO_TYPE-C-31-M-12, F.Cu at (100.3, 26.0)
- added J3: FH12A-12S-0.5SH(55), Connector_FFC-FPC:Hirose_FH12-12S-0.5SH_1x12-1MP_P0.50mm_Horizontal, F.Cu at (81.1, 25.9)
- added JP1: TERM, Jumper:SolderJumper-2_P1.3mm_Open_RoundedPad1.0x1.5mm, F.Cu at (82.6, 35.0)
- added L1: 22uH, Inductor_SMD:L_Changjiang_FNR6045S, F.Cu at (74.5, 50.2)
- added Q1: AO3400A, Package_TO_SOT_SMD:SOT-23, F.Cu at (73.5, 33.9)
- added R1: 100k, Resistor_SMD:R_0603_1608Metric, F.Cu at (89.0, 52.5)
- added R10: 10k, Resistor_SMD:R_0603_1608Metric, F.Cu at (86.0, 21.3)
- added R11: 27R, Resistor_SMD:R_1206_3216Metric, F.Cu at (73.5, 37.2)
- added R12: 100R, Resistor_SMD:R_0603_1608Metric, F.Cu at (86.0, 27.9)
- added R13: 10k, Resistor_SMD:R_0603_1608Metric, F.Cu at (89.2, 27.9)
- added R14: 5.1k, Resistor_SMD:R_0603_1608Metric, F.Cu at (92.5, 28.5)
- added R15: 5.1k, Resistor_SMD:R_0603_1608Metric, F.Cu at (92.5, 23.5)
- added R19: 10k, Resistor_SMD:R_0603_1608Metric, F.Cu at (80.3, 5.00)
- added R2: 15k, Resistor_SMD:R_0603_1608Metric, F.Cu at (89.0, 50.8)
- added R20: 1k, Resistor_SMD:R_0603_1608Metric, F.Cu at (67.3, 7.80)
- added R21: 10k, Resistor_SMD:R_0603_1608Metric, F.Cu at (86.0, 25.7)
- added R22: 10k, Resistor_SMD:R_0603_1608Metric, F.Cu at (80.3, 10.6)
- added R23: 1.5k, Resistor_SMD:R_0603_1608Metric, F.Cu at (27.5, 58.5)
- added R24: 3.3k, Resistor_SMD:R_0603_1608Metric, F.Cu at (40.5, 58.5)
- added R25: 6.8k, Resistor_SMD:R_0603_1608Metric, F.Cu at (53.5, 58.5)
- added R26: 1k, Resistor_SMD:R_0603_1608Metric, F.Cu at (67.3, 13.8)
- added R27: 1k, Resistor_SMD:R_0603_1608Metric, F.Cu at (67.3, 10.8)
- added R3: 100k, Resistor_SMD:R_0603_1608Metric, F.Cu at (89.0, 55.9)
- added R4: 13.3k, Resistor_SMD:R_0603_1608Metric, F.Cu at (89.0, 54.2)
- added R5: 120R DNP, Resistor_SMD:R_0603_1608Metric, F.Cu at (79.2, 35.0)
- added R6: 1k DNP, Resistor_SMD:R_0603_1608Metric, F.Cu at (78.4, 38.6)
- added R7: 1k DNP, Resistor_SMD:R_0603_1608Metric, F.Cu at (81.6, 38.6)
- added R8: 10k, Resistor_SMD:R_0603_1608Metric, F.Cu at (75.5, 7.60)
- added R9: 10k, Resistor_SMD:R_0603_1608Metric, F.Cu at (75.5, 10.4)
- added SW1: -, Button_Switch_SMD:SW_SPST_PTS645Sx43SMTR92, F.Cu at (14.5, 52.0)
- added SW2: +, Button_Switch_SMD:SW_SPST_PTS645Sx43SMTR92, F.Cu at (27.5, 52.0)
- added SW3: OK, Button_Switch_SMD:SW_SPST_PTS645Sx43SMTR92, F.Cu at (40.5, 52.0)
- added SW4: BACK, Button_Switch_SMD:SW_SPST_PTS645Sx43SMTR92, F.Cu at (53.5, 52.0)
- added TP1: EN, TestPoint:TestPoint_Pad_1.0x1.0mm, F.Cu at (75.5, 4.80)
- added TP2: BOOT, TestPoint:TestPoint_Pad_1.0x1.0mm, F.Cu at (77.6, 13.0)
- added U1: ESP32-C3-WROOM-02-N4, RF_Module:ESP32-C3-WROOM-02, F.Cu at (92.0, 7.10)
- added U2: TPS54202DDC, Package_TO_SOT_SMD:SOT-23-6, F.Cu at (83.5, 50.2)
- added U3: ME6211C33M5G-N, Package_TO_SOT_SMD:SOT-23-5, F.Cu at (69.0, 43.5)
- added U4: THVD1400DR, Package_SO:SOIC-8_3.9x4.9mm_P1.27mm, F.Cu at (82.5, 42.8)
Routing:
- net /BTN_ADC: track 0.00 -> 128.4 mm, vias 0 -> 3
- net +3V3: track 0.00 -> 88.9 mm
- net /RS485_TX: track 0.00 -> 68.9 mm, vias 0 -> 3
- net +5V: track 0.00 -> 66.3 mm, vias 0 -> 4
- net /RS485_DE: track 0.00 -> 62.2 mm, vias 0 -> 3
- net /RS485_RX: track 0.00 -> 48.8 mm, vias 0 -> 2
- net GND: track 0.00 -> 44.9 mm, vias 0 -> 34
- net Net-(U1-IO20/RXD): track 0.00 -> 44.1 mm, vias 0 -> 2
- net /TFT_SCK: track 0.00 -> 41.4 mm, vias 0 -> 2
- net /TFT_CS: track 0.00 -> 39.2 mm, vias 0 -> 2
- net /TFT_MOSI: track 0.00 -> 36.4 mm, vias 0 -> 2
- net Net-(U1-IO10): track 0.00 -> 36.1 mm, vias 0 -> 2
- net /TFT_DC: track 0.00 -> 36.1 mm
- net /RS485_A: track 0.00 -> 32.7 mm, vias 0 -> 4
- net /TFT_BL_PWM: track 0.00 -> 31.3 mm, vias 0 -> 2
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- added copper zone on B.Cu, net GND
- added copper zone on F.Cu, net GND
Other:
- board outline added: 104 x 66 mm
- copper layers 0 -> 2
- board text added: "+"
- board text added: "-"
- board text added: "A"
- board text added: "B"
- board text added: "BACK"
- board text added: "BUS"
- board text added: "DS1 glass rests on the board. Tail contacts face the viewer; J3 is a TOP-contact FH12A facing the glass, tail straight, entry face 16.9 mm from the glass edge (x 76.7). Keep the tail path (y 23-29, x 60-77) below 0.8 mm."
- board text added: "FAULT"
- board text added: "Keep enclosure metal >= 15 mm from the antenna."
- board text added: "M"
- board text added: "OK"
- board text added: "PWR"
- board text added: "U1 antenna overhangs the board edge by 6 mm (Espressif HDG preferred position)."
- board text added: "VALLOX RS-485 CONTROLLER rev A"
- board text added: "mironet.fi github.com/Miroeilola/vallox-rs485-controller"
